File: Module1/Electronics/module.sch (KiCad schematic (older format))
At the start: 13 parts

Commit message: ready for test, prototype
Parts:
- R?: value R -> 1
- R?: value R -> 10
- R?: value R -> 180
- R?: value R -> 1k
- R?: value R -> 10k
- R?: value R -> 100k
Changed lines of the file:
@@
 P 4400 5800
 F 0 "R?" V 4480 5800 50  0000 C CNN
-F 1 "R" V 4400 5800 50  0000 C CNN
+F 1 "1" V 4400 5800 50  0000 C CNN
 F 2 "" V 4330 5800 50  0000 C CNN
 F 3 "" H 4400 5800 50  0000 C CNN
@@
 P 4400 5950
 F 0 "R?" V 4480 5950 50  0000 C CNN
-F 1 "R" V 4400 5950 50  0000 C CNN
+F 1 "10" V 4400 5950 50  0000 C CNN
 F 2 "" V 4330 5950 50  0000 C CNN
 F 3 "" H 4400 5950 50  0000 C CNN
@@
 P 4400 6100
 F 0 "R?" V 4480 6100 50  0000 C CNN
-F 1 "R" V 4400 6100 50  0000 C CNN
+F 1 "180" V 4400 6100 50  0000 C CNN
 F 2 "" V 4330 6100 50  0000 C CNN
 F 3 "" H 4400 6100 50  0000 C CNN
@@
 P 4400 6250
 F 0 "R?" V 4480 6250 50  0000 C CNN
-F 1 "R" V 4400 6250 50  0000 C CNN
+F 1 "1k" V 4400 6250 50  0000 C CNN
 F 2 "" V 4330 6250 50  0000 C CNN
 F 3 "" H 4400 6250 50  0000 C CNN
@@
 P 4400 6400
 F 0 "R?" V 4480 6400 50  0000 C CNN
-F 1 "R" V 4400 6400 50  0000 C CNN
+F 1 "10k" V 4400 6400 50  0000 C CNN
 F 2 "" V 4330 6400 50  0000 C CNN
 F 3 "" H 4400 6400 50  0000 C CNN
@@
 P 4400 6550
 F 0 "R?" V 4480 6550 50  0000 C CNN
-F 1 "R" V 4400 6550 50  0000 C CNN
+F 1 "100k" V 4400 6550 50  0000 C CNN
 F 2 "" V 4330 6550 50  0000 C CNN
 F 3 "" H 4400 6550 50  0000 C CNN
